Commit message: changes for uav marker position

File: urdf/qr_mark.urdf.xacro (robot description, xacro)
@@ -16,5 +16,5 @@
         <origin xyz="-0.0 -0.04 0.04" rpy="-1.570796327 0 0" />
         <geometry>
-            <mesh filename="package://ed_pmov/meshes/25h09_0/meshes/25h09_0.dae" scale="0.25 0.2 0.2"/> <!--qrb.dae-->
+            <mesh filename="package://ed_pmov/meshes/25h09_0/meshes/25h09_0.dae" scale="0.35 0.3 0.3"/> <!--qrb.dae-->
         </geometry>
       </visual>
@@ -22,10 +22,10 @@
         <origin xyz="-0.0 0 -0.0" rpy="-1.570796327 0 0 " />
         <geometry>
-	    <mesh filename="package://ed_pmov/meshes/25h09_0/meshes/25h09_0.dae" scale="0.25 0.2 0.2"/>
+	    <mesh filename="package://ed_pmov/meshes/25h09_0/meshes/25h09_0.dae" scale="0.35 0.3 0.3"/>
         </geometry>
       </collision>
     </link>
   <joint name="${name}_joint1" type="fixed">
-     <origin xyz="0.15 0 -0.031" rpy="3.141592654  0 0" />
+     <origin xyz="0.16 0 -0.031" rpy="3.141592654  0 0" />
       <parent link="${parent}"/>
       <child link="${name}_link1"/>

File: urdf/quadrotor_base_mark.urdf.xacro (robot description, xacro)
@@ -30,5 +30,5 @@
     </xacro:sonar_sensor>
 		<xacro:qr_mark name="qr" parent="base_linkq" >
-    				  <origin xyz="0.055 0.04 -0.0" rpy="1.5708  1.5708 0"/>
+    				  <origin xyz="0.055 0.04 -0.05" rpy="1.5708 1.5708 1.0"/>
     		</xacro:qr_mark>
    <gazebo reference="base_linkq">

Commit message: fix eeff camera position for gazebo simmulation

File: urdf/qr_mark.urdf.xacro (robot description, xacro)
@@ -27,5 +27,5 @@
     </link>
   <joint name="${name}_joint1" type="fixed">
-     <origin xyz="0.16 0 -0.031" rpy="3.141592654  0 0" />
+     <origin xyz="0.18 0 -0.031" rpy="3.141592654  0 0" />
       <parent link="${parent}"/>
       <child link="${name}_link1"/>

File: urdf/quadrotor_base_mark.urdf.xacro (robot description, xacro)
@@ -30,5 +30,5 @@
     </xacro:sonar_sensor>
 		<xacro:qr_mark name="qr" parent="base_linkq" >
-    				  <origin xyz="0.055 0.04 -0.05" rpy="1.5708 1.5708 1.0"/>
+    				  <origin xyz="0.049 0.04 -0.01" rpy="1.5708 1.5708 0.0"/>
     		</xacro:qr_mark>
    <gazebo reference="base_linkq">
