Commit message: fixed partially world for simmulation

File: urdf/quadrotor_base_mark.urdf.xacro (robot description, xacro)
@@ -2,5 +2,6 @@
 <robot xmlns:xacro="http://www.ros.org/wiki/xacro">
   <xacro:include filename="$(find hector_sensors_description)/urdf/sonar_sensor.urdf.xacro" />
-<xacro:include filename="$(find ed_pmov)/urdf/qr_mark.urdf.xacro" />
+  <xacro:include filename="$(find ed_pmov)/urdf/qr_mark.urdf.xacro" />
+  <xacro:include filename="$(find ed_pmov)/urdf/quadrotor_camera.urdf.xacro" />
   <xacro:property name="pi" value="3.1415926535897931" />
   <!-- Main quadrotor link -->
@@ -25,11 +26,15 @@
       </collision>
     </link>
+    <!-- UAV camera sensor -->
+    <xacro:uav_camera parent="base_linkq">
+      <origin xyz="0.187 0.0 0.0183" rpy="0 0.4 0"/>
+    </xacro:uav_camera>
     <!-- Sonar height sensor -->
-    <xacro:sonar_sensor name="sonar" parent="base_linkq" ros_topic="sonar_height" update_rate="20" min_range="0.03" max_range="6.0" field_of_view="${30*pi/180}" ray_count="1">
-      <origin xyz="0.016 0.0 -0.01" rpy="0 ${90*pi/180} 0"/>
+    <xacro:sonar_sensor name="sonar" parent="base_linkq" ros_topic="sonar_height" update_rate="15" min_range="0.03" max_range="6.0" field_of_view="${30*pi/180}" ray_count="1">
+    	<origin xyz="-0.05 0.0 -0.01" rpy="0 ${90*pi/180} 0"/>
     </xacro:sonar_sensor>
-		<xacro:qr_mark name="qr" parent="base_linkq" >
-    				  <origin xyz="0.049 0.04 -0.01" rpy="1.5708 1.5708 0.0"/>
-    		</xacro:qr_mark>
+    <xacro:qr_mark name="qr" parent="base_linkq" >
+    	<origin xyz="0.04 0.04 -0.01" rpy="${pi/2} ${pi/2} 0.0"/>
+    </xacro:qr_mark>
    <gazebo reference="base_linkq">
      <gravity>true</gravity>
