Commit message: fixed world and urdf models

File: urdf/camera.urdf.xacro (robot description, xacro)
@@ -1,15 +1,14 @@
 <?xml version="1.0"?>
 <robot xmlns:xacro="http://www.ros.org/wiki/xacro">
-  <xacro:macro name="uav_camera" params="parent *origin ">
-<joint name="uav_cam_optical_joint" type="fixed">
+  <xacro:macro name="general_camera" params="name parent *origin ">
+<joint name="${name}_cam_optical_joint" type="fixed">
       <xacro:insert_block name="origin" />
       <parent link="${parent}"/>
-      <child link="uav_cam_optical_frame"/>
+      <child link="${name}_cam_optical_frame"/>
     </joint>
-    <link name="uav_cam_optical_frame"/>
-  </xacro:macro>
-	<gazebo reference="uav_cam_optical_frame">
+    <link name="${name}_cam_optical_frame"/>
+	<gazebo reference="${name}_cam_optical_frame">
 	       <turnGravityOff>true</turnGravityOff>
-		<sensor type="camera" name="cam_camera_sensor">
+		<sensor type="camera" name="${name}_camera_sensor">
 		  <update_rate>13.0</update_rate>
 		  <camera>
@@ -25,9 +24,9 @@
 		    </clip>
 		  </camera>
-		  <plugin name="cam_camera_controller" filename="libgazebo_ros_camera.so">
-		    <cameraName>uav_cam</cameraName>
+		  <plugin name="${name}_camera_controller" filename="libgazebo_ros_camera.so">
+		    <cameraName>${name}_cam</cameraName>
 		  <imageTopicName>image_raw</imageTopicName>
 		    <cameraInfoTopicName>camera_info</cameraInfoTopicName>
-		    <frameName>uav_cam_optical_frame</frameName>
+		    <frameName>${name}_cam_optical_frame</frameName>
 		  <hackBaseline>0.0</hackBaseline>
 		  <distortionK1>0.0</distortionK1>
@@ -39,3 +38,4 @@
 		</sensor>
 	</gazebo>
+</xacro:macro>
 </robot>

File: urdf/pioneer_with_proarm.urdf.xacro (robot description, xacro)
@@ -9,4 +9,5 @@
 	<!-- Import all available sensors -->
 	<xacro:include filename="$(find robotnik_sensors)/urdf/all_sensors.urdf.xacro" />
+  	<xacro:include filename="$(find ed_pmov)/urdf/camera.urdf.xacro" />
 	<xacro:include filename="$(find sick_scan)/urdf/sick_lms1xx.urdf.xacro" />
 	<!-- Camara simple
@@ -15,4 +16,8 @@
     <xacro:include filename="$(find arm)/urdf/dynamixel_pro_arm_macro.urdf" />
     <xacro:arg name="prefix" default="pioneer_proarm_"/>
+ <!-- UGV camera sensor -->
+    <xacro:general_camera parent="$(arg prefix)base_link" name="ugv">
+      <origin xyz="0.22 0.0 0.3" rpy="0 0.0 0"/>
+    </xacro:general_camera>
     <xacro:pioneer3dx prefix="$(arg prefix)"/>
   <xacro:pro_arm parent="$(arg prefix)base_link">

File: urdf/quadrotor_base_mark.urdf.xacro (robot description, xacro)
@@ -3,5 +3,5 @@
   <xacro:include filename="$(find hector_sensors_description)/urdf/sonar_sensor.urdf.xacro" />
   <xacro:include filename="$(find ed_pmov)/urdf/qr_mark.urdf.xacro" />
-  <xacro:include filename="$(find ed_pmov)/urdf/quadrotor_camera.urdf.xacro" />
+  <xacro:include filename="$(find ed_pmov)/urdf/camera.urdf.xacro" />
   <xacro:property name="pi" value="3.1415926535897931" />
   <!-- Main quadrotor link -->
@@ -27,7 +27,7 @@
     </link>
     <!-- UAV camera sensor -->
-    <xacro:uav_camera parent="base_linkq">
+    <xacro:general_camera parent="base_linkq" name="uav">
       <origin xyz="0.187 0.0 0.0183" rpy="0 0.4 0"/>
-    </xacro:uav_camera>
+    </xacro:general_camera>
     <!-- Sonar height sensor -->
     <xacro:sonar_sensor name="sonar" parent="base_linkq" ros_topic="sonar_height" update_rate="15" min_range="0.03" max_range="6.0" field_of_view="${30*pi/180}" ray_count="1">
