Commit message: fixed worlds and uav control

File: urdf/pioneer_with_proarm.urdf.xacro (robot description, xacro)
@@ -17,5 +17,5 @@
     <xacro:pioneer3dx prefix="$(arg prefix)"/>
   <xacro:pro_arm parent="$(arg prefix)base_link">
-    	<origin xyz="-0.0 0 0.24" /><!--slightly above pioneer plattform-->
+    	<origin xyz="-0.0 0 0.24"   rpy="0 0 1.57"/><!--slightly above pioneer plattform-->
     </xacro:pro_arm>
 <!--laser

Commit message: fixed for real robots and added world and controller config

File: urdf/pioneer_with_proarm.urdf.xacro (robot description, xacro)
@@ -14,5 +14,5 @@
  	 <xacro:include filename="$(find hector_sensors_description)/urdf/generic_camera.urdf.xacro" />
     	 <xacro:include filename="$(find hector_sensors_description)/urdf/asus_camera.urdf.xacro" />-->
-    <xacro:include filename="$(find arm)/urdf/dynamixel_pro_arm_macro.urdf" />
+    <xacro:include filename="$(find ed_pmov)/urdf/dynamixel_pro_arm_macro.urdf" />
     <xacro:arg name="prefix" default="pioneer_proarm_"/>
  <!-- UGV camera sensor -->
@@ -22,5 +22,5 @@
     <xacro:pioneer3dx prefix="$(arg prefix)"/>
   <xacro:pro_arm parent="$(arg prefix)base_link">
-    	<origin xyz="-0.0 0 0.24"   rpy="0 0 1.57"/><!--slightly above pioneer plattform-->
+    	<origin xyz="-0.0 0 0.26"   rpy="0 0 1.57"/><!--slightly above pioneer plattform-->
     </xacro:pro_arm>
 <!--laser
